File: AN021-Tracker-4-20mA-Quad/eagle/M8-Quad-420mA-Boost.sch (EAGLE design)
At the start: 30 parts, among them J1 CONN-B8B-M8, J2 TERMBLOCK-8X0.1, J3 TERMBLOCK-8X0.15, J4 TERMBLOCK-2X3.5MM, U1 MAX14626, U2 MAX14626, U3 MAX14626, U4 MAX14626, U5 XCL224, U6 ADS1015, U8 AP3012

Commit message: AN021
- Change value of sense resistor to 10 ohms
Parts:
- R1, R2, R3, R4: value 100 -> 10
Changed lines of the file:
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@@
 <part name="GND5" library="rickk2" deviceset="GND" device=""/>
 <part name="U1" library="rickk2" deviceset="MAX14626" device="" value="MAX14626"/>
-<part name="R1" library="rickk2" deviceset="RES-100-0603.DEV" device="" value="100"/>
+<part name="R1" library="rickk2" deviceset="RES-100-0603.DEV" device="" value="10"/>
 <part name="SUPPLY8" library="rickk2" deviceset="24V" device="" value="24V"/>
 <part name="D2" library="rickk2" deviceset="DIODE-TVS-SMAJ26A" device="" value="SMAJ26A"/>
 <part name="GND6" library="rickk2" deviceset="GND" device=""/>
 <part name="U2" library="rickk2" deviceset="MAX14626" device="" value="MAX14626"/>
-<part name="R2" library="rickk2" deviceset="RES-100-0603.DEV" device="" value="100"/>
+<part name="R2" library="rickk2" deviceset="RES-100-0603.DEV" device="" value="10"/>
 <part name="D3" library="rickk2" deviceset="DIODE-TVS-SMAJ26A" device="" value="SMAJ26A"/>
 <part name="GND7" library="rickk2" deviceset="GND" device=""/>
 <part name="U3" library="rickk2" deviceset="MAX14626" device="" value="MAX14626"/>
-<part name="R3" library="rickk2" deviceset="RES-100-0603.DEV" device="" value="100"/>
+<part name="R3" library="rickk2" deviceset="RES-100-0603.DEV" device="" value="10"/>
 <part name="D4" library="rickk2" deviceset="DIODE-TVS-SMAJ26A" device="" value="SMAJ26A"/>
 <part name="GND8" library="rickk2" deviceset="GND" device=""/>
 <part name="U4" library="rickk2" deviceset="MAX14626" device="" value="MAX14626"/>
-<part name="R4" library="rickk2" deviceset="RES-100-0603.DEV" device="" value="100"/>
+<part name="R4" library="rickk2" deviceset="RES-100-0603.DEV" device="" value="10"/>
 <part name="U8" library="rickk2" deviceset="AP3012" device="" value="AP3012"/>
 <part name="L2" library="rickk2" deviceset="INDUCTOR-10UH" device="" value="10uH"/>
